File: KiCad/TrackController/TrackController.kicad_pcb (KiCad board)
At the start: 2 copper layers, 133.5 x 74 mm, 3 parts, among them J1 DE9_Plug_MountingHoles, U1 mini ESP32, U2 TXS0108EPW

Commit message: Added KiCAD pcb design
Parts:
- added A1: Arduino_Uno_R3_Shield, PCM_arduino-library:Arduino_Uno_R3_Shield, F.Cu at (81.9, 126.7)
- added LCD1: ~, railtrack:1.77 LCD Display 128x160, B.Cu at (77.1, 94.0)
- added Q1: BC547, Package_TO_SOT_THT:TO-92_Inline, F.Cu at (47.6, 121.6)
- added Q2: BC547, Package_TO_SOT_THT:TO-92_Inline, F.Cu at (55.2, 121.6)
- added Q3: BC547, Package_TO_SOT_THT:TO-92_Inline, F.Cu at (62.9, 121.6)
- added SW1: SW_Push, Button_Switch_THT:SW_PUSH_6mm, B.Cu at (104.1, 120.0)
- added SW2: SW_Push, Button_Switch_THT:SW_PUSH_6mm, B.Cu at (110.6, 80.0)
- added U3: ~, railtrack:MCP2515 Module, F.Cu at (120.0, 100.0)
- added U4: ~, railtrack:MP1484 Module, F.Cu at (159.4, 116.5)
- U1: value mini ESP32 -> mini_esp32
- moved U2 49.5 mm to (84.0, 91.0)
- moved U1 47.6 mm to (61.6, 100.0), turned to -90 degrees
- moved J1 42.1 mm to (160.2, 94.1), turned to 90 degrees
Connections:
- U1 pad 1: (no net) -> GND
- U1 pad 10: (no net) -> unconnected-(U1-IO_19/D6-Pad10)
- U1 pad 11: (no net) -> unconnected-(U1-IO_34-Pad11)
- U1 pad 12: (no net) -> unconnected-(U1-IO_23/D7-Pad12)
- U1 pad 13: (no net) -> unconnected-(U1-IO_14/TMS-Pad13)
- U1 pad 14: (no net) -> unconnected-(U1-IO_05/D8-Pad14)
- U1 pad 15: (no net) -> unconnected-(U1-NC-Pad15)
- U1 pad 16: (no net) -> /3V3
- U1 pad 17: (no net) -> unconnected-(U1-IO_09/SD2-Pad17)
- U1 pad 18: (no net) -> unconnected-(U1-IO_13/TCK-Pad18)
- U1 pad 19: (no net) -> unconnected-(U1-CMD-Pad19)
- U1 pad 2: (no net) -> unconnected-(U1-RST-Pad2)
- U1 pad 20: (no net) -> unconnected-(U1-IO_10/SD3-Pad20)
- U1 pad 21: (no net) -> unconnected-(U1-TXD-Pad21)
- U1 pad 22: (no net) -> GND
- U1 pad 23: (no net) -> unconnected-(U1-RXD-Pad23)
- U1 pad 24: (no net) -> unconnected-(U1-IO_27-Pad24)
- U1 pad 25: (no net) -> unconnected-(U1-IO_22/D1/SCL-Pad25)
- U1 pad 26: (no net) -> unconnected-(U1-IO_25-Pad26)
- U1 pad 27: (no net) -> unconnected-(U1-IO_21/D2/SDA-Pad27)
- U1 pad 28: (no net) -> unconnected-(U1-IO_32-Pad28)
- U1 pad 29: (no net) -> unconnected-(U1-IO_17/D3-Pad29)
- U1 pad 3: (no net) -> unconnected-(U1-NC-Pad3)
- U1 pad 30: (no net) -> unconnected-(U1-IO_12/TDI-Pad30)
- U1 pad 31: (no net) -> unconnected-(U1-IO_16/D4-Pad31)
- U1 pad 32: (no net) -> unconnected-(U1-IO_04-Pad32)
- U1 pad 33: (no net) -> GND
- U1 pad 34: (no net) -> unconnected-(U1-IO_00-Pad34)
- U1 pad 35: (no net) -> /VCC
- U1 pad 36: (no net) -> unconnected-(U1-IO_02-Pad36)
- U1 pad 37: (no net) -> unconnected-(U1-TD0-Pad37)
- U1 pad 38: (no net) -> unconnected-(U1-SD1-Pad38)
- U1 pad 39: (no net) -> unconnected-(U1-SD0-Pad39)
- U1 pad 4: (no net) -> unconnected-(U1-IO_36/SVP/A0-Pad4)
- U1 pad 40: (no net) -> unconnected-(U1-CLK-Pad40)
- U1 pad 5: (no net) -> unconnected-(U1-IO_39/SVN-Pad5)
- U1 pad 6: (no net) -> unconnected-(U1-IO_26/D0-Pad6)
- U1 pad 7: (no net) -> unconnected-(U1-IO_35-Pad7)
- U1 pad 8: (no net) -> unconnected-(U1-IO_18/D5-Pad8)
- U1 pad 9: (no net) -> unconnected-(U1-IO_33-Pad9)
- U2 pad 11: unconnected-(U2-GND-Pad11) -> GND
- U2 pad 19: unconnected-(U2-VCCB-Pad19) -> /VCC
- U2 pad 2: unconnected-(U2-VCCA-Pad2) -> /3V3
Other:
- board size 133.5 x 74 mm -> 160 x 100 mm

Commit message: 20240422
Parts:
- removed A1: Arduino_Uno_R3_Shield, PCM_arduino-library:Arduino_Uno_R3_Shield
- removed Q1, Q2, Q3: BC547, Package_TO_SOT_THT:TO-92_Inline
- added R1: 10k, Resistor_THT:R_Axial_DIN0207_L6.3mm_D2.5mm_P7.62mm_Horizontal, F.Cu at (50.4, 73.5)
- added U5: ~, railtrack:Arduino_Shield, F.Cu at (81.7, 126.7)
- added U6: ~, railtrack:IBT_2, F.Cu at (53.1, 79.7)
Connections:
- J1 pad 0: unconnected-(J1-PAD-Pad0) -> GND
- J1 pad 1: unconnected-(J1-Pad1) -> GND
- J1 pad 3: unconnected-(J1-Pad3) -> /CAN-H
- J1 pad 5: unconnected-(J1-Pad5) -> /CAN-L
- J1 pad 9: unconnected-(J1-Pad9) -> /18V
- LCD1 pad 2: unconnected-(LCD1-VCC-Pad2) -> /VCC
- LCD1 pad 3: unconnected-(LCD1-SCL-Pad3) -> /SCK
- LCD1 pad 4: unconnected-(LCD1-SDA-Pad4) -> /MOSI
- LCD1 pad 5: unconnected-(LCD1-RES-Pad5) -> /LCD-RES
- LCD1 pad 6: unconnected-(LCD1-RS-Pad6) -> /LCD-RS
- LCD1 pad 7: unconnected-(LCD1-CS-Pad7) -> /LCD-CS*
- LCD1 pad 8: unconnected-(LCD1-LED_A-Pad8) -> /3V3
- SW1 pad 1: unconnected-(SW1-Pad1) -> GND
- SW1 pad 2: unconnected-(SW1-Pad2) -> /MEASUREMENT_TOGGLE
- SW2 pad 1: unconnected-(SW2-Pad1) -> GND
- U1 pad 10: unconnected-(U1-IO_19/D6-Pad10) -> /MISO
- U1 pad 11: unconnected-(U1-IO_34-Pad11) -> /IS
- U1 pad 12: unconnected-(U1-IO_23/D7-Pad12) -> /MOSI
- U1 pad 14: unconnected-(U1-IO_05/D8-Pad14) -> /CAN-CS*
- U1 pad 24: unconnected-(U1-IO_27-Pad24) -> /MEASUREMENT_TOGGLE
- U1 pad 25: unconnected-(U1-IO_22/D1/SCL-Pad25) -> /CAN-INT*
- U1 pad 26: unconnected-(U1-IO_25-Pad26) -> /TRACK-POWER-ENABLE
- U1 pad 27: unconnected-(U1-IO_21/D2/SDA-Pad27) -> /LCD-RS
- U1 pad 28: unconnected-(U1-IO_32-Pad28) -> /TRACK-PULSE-H
- U1 pad 29: unconnected-(U1-IO_17/D3-Pad29) -> /LCD-RES
- U1 pad 31: unconnected-(U1-IO_16/D4-Pad31) -> /LCD-CS*
- U1 pad 5: unconnected-(U1-IO_39/SVN-Pad5) -> /VOLTAGE
- U1 pad 7: unconnected-(U1-IO_35-Pad7) -> /TEMP
- U1 pad 8: unconnected-(U1-IO_18/D5-Pad8) -> /SCK
- U1 pad 9: unconnected-(U1-IO_33-Pad9) -> /TRACK-PULSE-L
- U2 pad 1: unconnected-(U2-A1-Pad1) -> /SCK
- U2 pad 15: unconnected-(U2-B5-Pad15) -> /CAN-INT-TTL*
- U2 pad 16: unconnected-(U2-B4-Pad16) -> /CAN-CS-TTL*
- U2 pad 17: unconnected-(U2-B3-Pad17) -> /SO-TTL
- U2 pad 18: unconnected-(U2-B2-Pad18) -> /SI-TTL
- U2 pad 20: unconnected-(U2-B1-Pad20) -> /SCK-TTL
- U2 pad 3: unconnected-(U2-A2-Pad3) -> /MOSI
- U2 pad 4: unconnected-(U2-A3-Pad4) -> /MISO
- U2 pad 5: unconnected-(U2-A4-Pad5) -> /CAN-CS*
- U2 pad 6: unconnected-(U2-A5-Pad6) -> /CAN-INT*
- U3 pad 1: unconnected-(U3-INT-Pad1) -> /CAN-INT-TTL*
- U3 pad 2: unconnected-(U3-SCK-Pad2) -> /SCK-TTL
- U3 pad 3: unconnected-(U3-SI-Pad3) -> /SI-TTL
- U3 pad 4: unconnected-(U3-SO-Pad4) -> /SO-TTL
- U3 pad 5: unconnected-(U3-CS-Pad5) -> /CAN-CS-TTL*
- U3 pad 7: unconnected-(U3-VCC-Pad7) -> /VCC
- U3 pad 8: unconnected-(U3-CAN-H-Pad8) -> /CAN-H
- U3 pad 9: unconnected-(U3-CAN-L-Pad9) -> /CAN-L
- U4 pad 7: /VCC -> /VCC-RAW
- U4 pad 8: /VCC -> /VCC-RAW
Routing:
- net /VCC: track 0.00 -> 25.5 mm
- net /SO-TTL: track 0.00 -> 14.0 mm
- net /CAN-INT-TTL*: track 0.00 -> 11.1 mm
- added copper zone on F.Cu, net GND

Commit message: 20240423
Parts:
- added J3: Barrel_Jack_Switch, Connector_BarrelJack:BarrelJack_CUI_PJ-102AH_Horizontal, F.Cu at (53.2, 123.2)
- added JP1: Jumper_2_Open, Jumper:SolderJumper-2_P1.3mm_Open_TrianglePad1.0x1.5mm, F.Cu at (147.3, 119.0)
- moved R1 57.7 mm to (75.6, 125.4), turned to 90 degrees
- moved U6 43.6 mm to (65.4, 121.6)
- moved SW1 29.3 mm to (132.8, 114.2)
- moved SW2 28.7 mm to (139.0, 84.0)
- moved LCD1 28.5 mm to (105.0, 100.0), turned to 0 degrees
- moved U3 6.35 mm to (126.4, 100.0)
- moved U2 6.00 mm to (90.0, 91.0)
- moved U1 3.81 mm to (57.8, 100.0)
- moved J1 1.98 mm to (162.2, 93.7)
Connections:
- SW2 pad 2: unconnected-(SW2-Pad2) -> /SPARE-SWITCH
- U1 pad 6: unconnected-(U1-IO_26/D0-Pad6) -> /SPARE-SWITCH
- U2 pad 10: unconnected-(U2-OE-Pad10) -> /3V3
- U2 pad 12: unconnected-(U2-B8-Pad12) -> /TRACK-PULSE-H-PROG-TTL
- U2 pad 13: unconnected-(U2-B7-Pad13) -> /TRACK-PULSE-H-TTL
- U2 pad 14: unconnected-(U2-B6-Pad14) -> /TRACK-ENABLE-TTL
- U2 pad 7: unconnected-(U2-A6-Pad7) -> /TRACK-POWER-ENABLE
- U2 pad 8: unconnected-(U2-A7-Pad8) -> /TRACK-PULSE-H
- U2 pad 9: unconnected-(U2-A8-Pad9) -> /TRACK-PULSE-H-PROG
- U5 pad J1-3: GND -> unconnected-(U5-AREF-PadJ1-3)
- U5 pad J1-4: (no net) -> GND
- U5 pad J1-5: unconnected-(U5-DIR-B-PadJ1-5) -> /TRACK-PULSE-H-PROG-TTL
- U5 pad J1-6: unconnected-(U5-DIR-A-PadJ1-6) -> /TRACK-PULSE-H-PROG
- U5 pad J1-7: unconnected-(U5-PWM-B-PadJ1-7) -> /TRACK-ENABLE-TTL
- U5 pad J1-9: (no net) -> unconnected-(U5-BREAK-A-PadJ1-9)
- U5 pad J2-5: unconnected-(U5-PWM-A-PadJ2-5) -> /TRACK-ENABLE-TTL
- U5 pad J4-1: unconnected-(U5-SENSE-A-PadJ4-1) -> /IS
- U6 pad 5: /iS -> /IS
Routing:
- net /SCK: track 0.00 -> 54.5 mm
- net /MOSI: track 0.00 -> 28.2 mm
- net /VCC: track 25.5 -> 0.00 mm, vias 0 -> 1
- net /SO-TTL: track 14.0 -> 0.00 mm
- net /CAN-INT-TTL*: track 11.1 -> 0.00 mm
- added copper zone on B.Cu, net GND
- removed copper zone on F.Cu, net GND
Other:
- board size 160 x 100 mm -> 130 x 60 mm

Commit message: 20240423
Parts:
- added R2: 100k, Resistor_THT:R_Axial_DIN0207_L6.3mm_D2.5mm_P7.62mm_Horizontal, F.Cu at (81.9, 126.0)
- added R3: 10k, Resistor_THT:R_Axial_DIN0207_L6.3mm_D2.5mm_P7.62mm_Horizontal, F.Cu at (88.3, 126.0)
- moved R1 0.63 mm to (75.6, 126.0)
Connections:
- U5 pad J4-3: unconnected-(U5-A2-PadJ4-3) -> /TEMP

Commit message: 20240423
Parts:
- moved R3 7.65 mm to (87.6, 118.4), turned to -90 degrees
Connections:
- U1 pad 2: unconnected-(U1-RST-Pad2) -> /RESET*
- U5 pad J3-3: unconnected-(U5-IOREF-PadJ3-3) -> /RESET*
Routing:
- net /18V: track 0.00 -> 141.2 mm
- net /TEMP: track 0.00 -> 133.4 mm
- net /IS: track 0.00 -> 130.4 mm
- net /VCC: track 0.00 -> 129.8 mm, vias 1 -> 0
- net /3V3: track 0.00 -> 125.0 mm
- net /VOLTAGE: track 0.00 -> 88.9 mm
- net /SPARE-SWITCH: track 0.00 -> 75.9 mm
- net /MEASUREMENT_TOGGLE: track 0.00 -> 74.3 mm
- net /RESET*: track 0.00 -> 69.5 mm
- net /TRACK-ENABLE-TTL: track 0.00 -> 57.2 mm
- net /TRACK-PULSE-H-PROG: track 0.00 -> 52.4 mm, vias 0 -> 1
- net /TRACK-PULSE-H: track 0.00 -> 41.5 mm
- net /TRACK-PULSE-L: track 0.00 -> 41.0 mm
- net /CAN-CS*: track 0.00 -> 40.2 mm
- net /TRACK-POWER-ENABLE: track 0.00 -> 39.5 mm
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