File: KiCad/TrackController/TrackController.kicad_pcb (KiCad board)
At the start: 2 copper layers, 130 x 60 mm, 15 parts, among them J1 DE9_Plug_MountingHoles, J3 Barrel_Jack_Switch, SW1 SW_Push, SW2 SW_Push, U1 mini_esp32, U2 TXS0108EPW

Commit message: 20240425
Parts:
- added C2: 100nF, Capacitor_THT:C_Disc_D5.1mm_W3.2mm_P5.00mm, F.Cu at (67.9, 120.3)
- added C4: 100nF, Capacitor_THT:C_Disc_D5.1mm_W3.2mm_P5.00mm, F.Cu at (139.0, 119.0)
- added CP1: 100uF/25V, Capacitor_THT:CP_Radial_D8.0mm_P5.00mm, F.Cu at (59.7, 120.3)
- added CP3: 100uF/25V, Capacitor_THT:CP_Radial_D8.0mm_P5.00mm, F.Cu at (145.9, 115.9)
- added G***: LOGO, LOGO, B.Cu at (159.4, 116.5)
- added G1: LOGO, LOGO, F.Cu at (155.1, 85.0)
- added SW3: SW_Push, Button_Switch_THT:SW_PUSH_6mm, B.Cu at (141.0, 102.1)
- added SW4: SW_Push, Button_Switch_THT:SW_PUSH_6mm, B.Cu at (141.0, 111.0)
- added U3: ~, Package_TO_SOT_THT:TO-92, F.Cu at (102.2, 122.2)
- J3: footprint Connector_BarrelJack:BarrelJack_CUI_PJ-102AH_Horizontal -> Connector_BarrelJack:BarrelJack_GCT_DCJ200-10-A_Horizontal
- JP1: footprint Jumper:SolderJumper-2_P1.3mm_Open_TrianglePad1.0x1.5mm -> Connector_PinHeader_2.54mm:PinHeader_1x02_P2.54mm_Vertical
- moved SW1 30.9 mm to (141.0, 84.4), turned to 180 degrees
- moved IBT_2 26.7 mm to (92.1, 122.2)
- moved JP1 18.4 mm to (128.9, 119.0), turned to -90 degrees
- moved SW2 9.54 mm to (141.0, 93.3)
- moved R3 7.01 mm to (80.6, 119.0)
- moved R2 5.07 mm to (76.8, 126.7)
- moved R1 2.62 mm to (73.0, 126.7)
- renumbered U3 to CAN-MODULE1, U1 to ESP32, U6 to IBT_2, U5 to MOTOR-SHIELD1, U2 to U1, U4 to U2
Connections:
- net /SPARE-SWITCH renamed /SPARE-SWITCH-1
- ESP32 pad 4: unconnected-(U1-IO_36/SVP/A0-Pad4) -> /SPARE-SWITCH-2
Routing:
- net /SPARE-SWITCH-2: track 0.00 -> 98.8 mm
- net /VCC: track 129.8 -> 177.9 mm
- net /VOLTAGE: track 88.9 -> 46.1 mm
- net /RESET*: track 69.5 -> 102.6 mm, vias 0 -> 1
- net /TRACK-PULSE-L: track 41.0 -> 72.3 mm
- net /SPARE-SWITCH-1: track 75.9 -> 102.8 mm
- net /TEMP: track 133.4 -> 107.4 mm, vias 0 -> 1
- net /VCC-RAW: track 11.4 -> 30.0 mm
- net /IS: track 130.4 -> 113.8 mm
- net /3V3: track 125.0 -> 111.8 mm
- net /TRACK-POWER-ENABLE: track 39.5 -> 50.5 mm
- net /MOSI: track 50.5 -> 39.8 mm
- net /SCK: track 44.3 -> 33.7 mm
- net /MEASUREMENT_TOGGLE: track 74.3 -> 84.7 mm, vias 0 -> 1
- net /TRACK-PULSE-H-PROG: track 52.4 -> 43.0 mm, vias 1 -> 0
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- added copper zone on F.Cu, net GND
Other:
- outline, holes or cut-outs redrawn
- board text added: "Adjust MP1584 to 5V before closing pins"
- board text added: "DCC-Railtrack controller Marklin-CAN Bridge https://github.com/GerardHarkema/railtrack/ Design by Gerard Harkema(2024/04/26)"
- board text added: "RESET"
- board text added: "SPARE-1"
- board text added: "SPARE2"
- board text added: "TOGGLE-MEASUREMENT"
