File: KiCad/TrackController/TrackController.kicad_sch (KiCad schematic)
At the start: 3 parts, among them J1 DE9_Plug_MountingHoles, U1 mini_esp32, U2 TXS0108EPW

Commit message: Added KiCAD pcb design
Parts:
- added A1: Arduino_Uno_R3_Shield, PCM_arduino-library:Arduino_Uno_R3_Shield, symbol PCM_arduino-library:Arduino_Uno_R3_Shield
- added J3: Barrel_Jack_Switch, symbol Connector:Barrel_Jack_Switch
- added LCD1: ~, railtrack:1.77 LCD Display 128x160, symbol railtrack:1.77_LCD_Display
- added Q1, Q2, Q3: BC547, Package_TO_SOT_THT:TO-92_Inline, symbol Transistor_BJT:BC547
- added SW1, SW2: SW_Push, Button_Switch_THT:SW_PUSH_6mm, symbol Switch:SW_Push
- added U3: ~, railtrack:MCP2515 Module, symbol railtrack:MCP2515_Module
- added U4: ~, railtrack:MP1484 Module, symbol railtrack:MP1585_module
- U1: footprint (none) -> ESP32_mini:ESP32_mini
Connections:
- net GND: now reaches U1.1 (GND)
- net GND: now also U1.22 (GND), U1.33 (GND), U2.11 (GND), A1.GND1 (GND), A1.GND2 (GND), A1.GND3 (GND), J3.2, J3.3, LCD1.1 (GND), Q1.3 (E), Q2.3 (E), Q3.3 (E), U3.6 (GND), U4.1 (GND), U4.2 (GND), U4.5 (GND), U4.6 (GND)
- net 3V3: now reaches U1.16 (3V3)
- net 3V3: now also U2.2 (VCCA), A1.3V3 (3.3V), LCD1.8 (LED_A)
- net VCC: now reaches U1.35 (VCC_(USB))
- net VCC: now also U2.19 (VCCB), A1.5V1 (5V), LCD1.2 (VCC), U4.7 (V-OUT), U4.8 (V-OUT)
- new net 18V: J3.1, U4.3 (V-IN), U4.4 (V-IN)
- new net CAN-CS-TTL*: U3.5 (CS)
- new net CAN-H: U3.8 (CAN-H)
- new net CAN-INT-TTL*: U3.1 (INT)
- new net CAN-L: U3.9 (CAN-L)
- new net LCD-CS*: LCD1.7 (CS)
- new net LCD-RES: LCD1.5 (RES)
- new net LCD-RS: LCD1.6 (RS)
- new net SCK-TTL: U3.2 (SCK)
- new net SCL: LCD1.3 (SCL)
- new net SDA: LCD1.4 (SDA)
- new net SI-TTL: U3.3 (SI)
- new net SO-TTL: U3.4 (SO)
Other:
- moved on the sheet: J1

Commit message: 20240422
Parts:
- removed A1: Arduino_Uno_R3_Shield, PCM_arduino-library:Arduino_Uno_R3_Shield, symbol PCM_arduino-library:Arduino_Uno_R3_Shield
- removed Q1, Q2, Q3: BC547, Package_TO_SOT_THT:TO-92_Inline, symbol Transistor_BJT:BC547
- added R1: 10k, Resistor_THT:R_Axial_DIN0207_L6.3mm_D2.5mm_P7.62mm_Horizontal, symbol Device:R
- added U5: ~, railtrack:Arduino_Shield, symbol railtrack:ARDUIN-MOTOR--SHIELD-REVB
- added U6: ~, railtrack:IBT_2, symbol railtrack:IBT_2
Connections:
- net SCL is gone; now on net SCK: LCD1.3 (SCL)
- net SDA is gone; now on net MOSI: LCD1.4 (SDA)
- net 18V: now also J1.9, U5.J3-8 (+18V), U6.9 (+18)
- net 3V3: now also U5.J3-4 (3V3), U6.8 (VCC)
- net CAN-CS-TTL*: now also U2.16 (B4)
- net CAN-H: now also J1.3
- net CAN-INT-TTL*: now also U2.15 (B5)
- net CAN-L: now also J1.5
- net GND: now also J1.0 (PAD), J1.1, SW1.1, SW2.1, R1.2, U5.J1-3 (GND), U5.J3-6 (GND), U5.J3-7 (GND), U6.7 (GND)
- net LCD-CS*: now also U1.31 (IO_16/D4)
- net LCD-RES: now also U1.29 (IO_17/D3)
- net LCD-RS: now also U1.27 (IO_21/D2/SDA)
- net SCK-TTL: now also U2.20 (B1)
- net SI-TTL: now also U2.18 (B2)
- net SO-TTL: now also U2.17 (B3)
- net VCC: now also U3.7 (VCC), U5.J3-5 (VCC); no longer U4.7 (V-OUT), U4.8 (V-OUT)
- net MEASUREMENT_TOGGLE: now reaches SW1.2
- net MEASUREMENT_TOGGLE: now also U1.24 (IO_27)
- net SCK: now reaches U2.1 (A1)
- net SCK: now also U1.8 (IO_18/D5)
- net MOSI: now reaches U2.3 (A2)
- net MOSI: now also U1.12 (IO_23/D7)
- net MISO: now reaches U2.4 (A3)
- net MISO: now also U1.10 (IO_19/D6)
- net CAN-CS*: now reaches U2.5 (A4)
- net CAN-CS*: now also U1.14 (IO_05/D8)
- net CAN-INT*: now reaches U2.6 (A5)
- net CAN-INT*: now also U1.25 (IO_22/D1/SCL)
- net IS: now reaches U1.11 (IO_34)
- net IS: now also R1.1, U6.6 (R-IS)
- net TRACK-POWER-ENABLE: now reaches U1.26 (IO_25)
- net TRACK-POWER-ENABLE: now also U6.3 (L-EN), U6.4 (R-EN)
- net TRACK-PULSE-H: now reaches U1.28 (IO_32)
- net TRACK-PULSE-H: now also U6.1 (L-PWM)
- net VOLTAGE: now reaches U1.5 (IO_39/SVN)
- net TEMP: now reaches U1.7 (IO_35)
- net TEMP: now also U6.10 (TEMP)
- net TRACK-PULSE-L: now reaches U1.9 (IO_33)
- net TRACK-PULSE-L: now also U6.2 (R-PWM)
- new net VCC-RAW: U4.7 (V-OUT), U4.8 (V-OUT)
- new net iS: U6.5 (L-IS)

Commit message: 20240423
Parts:
- added JP1: Jumper_2_Open, Jumper:SolderJumper-2_P1.3mm_Open_TrianglePad1.0x1.5mm, symbol Jumper:Jumper_2_Open
- J3: footprint (none) -> Connector_BarrelJack:BarrelJack_CUI_PJ-102AH_Horizontal
Connections:
- net iS is gone; now on net IS: U6.5 (L-IS)
- net 3V3: now also U2.10 (OE)
- net GND: now also U5.J1-4 (GND); no longer U5.J1-3 (GND)
- net IS: now also U5.J4-1 (SENSE-A)
- net TRACK-POWER-ENABLE: now also U2.7 (A6)
- net TRACK-PULSE-H: now also U2.8 (A7)
- net VCC: now also JP1.2 (B)
- net VCC-RAW: now also JP1.1 (A)
- net TRACK-PULSE-H-PROG-TTL: now reaches U5.J1-5 (DIR-B)
- net TRACK-PULSE-H-PROG-TTL: now also U2.12 (B8)
- net TRACK-PULSE-H-PROG: now reaches U5.J1-6 (DIR-A)
- net TRACK-PULSE-H-PROG: now also U2.9 (A8)
- net TRACK-ENABLE-TTL: now reaches U5.J1-7 (PWM-B)
- net TRACK-ENABLE-TTL: now also U2.14 (B6), U5.J2-5 (PWM-A)
- net TRACK-PULSE-H-TTL: now reaches U2.13 (B7)
- net SPARE-SWITCH: now reaches SW2.2
- net SPARE-SWITCH: now also U1.6 (IO_26/D0)

Commit message: 20240423
Parts:
- added R2: 100k, Resistor_THT:R_Axial_DIN0207_L6.3mm_D2.5mm_P7.62mm_Horizontal, symbol Device:R
- added R3: 10k, Resistor_THT:R_Axial_DIN0207_L6.3mm_D2.5mm_P7.62mm_Horizontal, symbol Device:R
Connections:
- net 18V: now also R2.1
- net GND: now also R3.2
- net TEMP: now also U5.J4-3 (A2)
- net VOLTAGE: now also R2.2, R3.1

Commit message: 20240423
Connections:
- net RESET*: now reaches U5.J3-3 (RESET)
- net RESET*: now also U1.2 (RST)
Changed lines of the file:
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@@
 	(wire
 		(pts
-			(xy 134.62 38.1) (xy 140.97 38.1)
+			(xy 134.62 38.1) (xy 143.51 38.1)
 		)
 		(stroke
@@
 		)
 	)
+	(label "RESET*"
+		(at 134.62 43.18 0)
+		(fields_autoplaced yes)
+		(effects
+			(font
+				(size 1.27 1.27)
+			)
+			(justify left bottom)
+		)
+	)
 	(label "SCK-TTL"
 		(at 182.88 38.1 0)
@@
 			)
 			(justify left bottom)
+		)
+	)
+	(label "RESET*"
+		(at 35.56 41.91 180)
+		(fields_autoplaced yes)
+		(effects
+			(font
+				(size 1.27 1.27)
+			)
+			(justify right bottom)
 		)
 	)
@@
 	(symbol
 		(lib_id "power:GND")
-		(at 140.97 38.1 0)
+		(at 143.51 38.1 0)
 		(unit 1)
 		(exclude_from_sim no)
@@
 		(fields_autoplaced yes)
 		(property "Reference" "#PWR05"
-			(at 140.97 44.45 0)
+			(at 143.51 44.45 0)
 			(effects
 				(font
@@
 		)
 		(property "Value" "GND"
-			(at 140.97 43.18 0)
+			(at 143.51 43.18 0)
 			(effects
 				(font
@@
 		)
 		(property "Footprint" ""
-			(at 140.97 38.1 0)
+			(at 143.51 38.1 0)
 			(effects
 				(font
@@
 		)
 		(property "Datasheet" ""
-			(at 140.97 38.1 0)
+			(at 143.51 38.1 0)
 			(effects
 				(font
@@
 		)
 		(property "Description" "Power symbol creates a global label with name \"GND\" , ground"
-			(at 140.97 38.1 0)
-			(effects
-				(font
+			(at 143.51 38.1 0)
+			(effects
+				(font
