File: KiCad/TrackController/TrackController.kicad_sch (KiCad schematic)
At the start: 15 parts, among them J1 DE9_Plug_MountingHoles, J3 Barrel_Jack_Switch, SW1 SW_Push, SW2 SW_Push, U1 mini_esp32, U2 TXS0108EPW

Commit message: 20240425
Parts:
- added C2, C4: 100nF, Capacitor_THT:C_Disc_D5.1mm_W3.2mm_P5.00mm, symbol Device:C
- added CP1, CP3: 100uF/25V, Capacitor_THT:CP_Radial_D8.0mm_P5.00mm, symbol Device:C_Polarized
- added SW3, SW4: SW_Push, Button_Switch_THT:SW_PUSH_6mm, symbol Switch:SW_Push
- added U3: ~, Package_TO_SOT_THT:TO-92, symbol railtrack:TMP36
- J3: footprint Connector_BarrelJack:BarrelJack_CUI_PJ-102AH_Horizontal -> Connector_BarrelJack:BarrelJack_GCT_DCJ200-10-A_Horizontal
- JP1: footprint Jumper:SolderJumper-2_P1.3mm_Open_TrianglePad1.0x1.5mm -> Connector_PinHeader_2.54mm:PinHeader_1x02_P2.54mm_Vertical
- renumbered U3 to CAN-MODULE1, U1 to ESP32, U6 to IBT_2, U5 to MOTOR-SHIELD1, U2 to U1, U4 to U2
Connections:
- net 18V: now also C2.1, CP1.1
- net GND: now also C2.2, C4.2, CP1.2, CP3.2, SW3.1, SW4.1, U3.3 (GND)
- net RESET*: now also SW4.2
- net TEMP: now also U3.2 (Temp)
- net VCC: now also C4.1, CP3.1, U3.1 (VCC)
- net SPARE-SWITCH-2: now reaches ESP32.4 (IO_36/SVP/A0)
- net SPARE-SWITCH-2: now also SW3.2
- net SPARE-SWITCH renamed SPARE-SWITCH-1
